Commit message: code dump

File: sam_bot_description/models/basic_mobile_bot_v1.urdf (robot description, URDF)
Before this commit: robot basic_mobile_bot, 5 links, 4 joints
Links:
- link base_link: geometry collision box size=${base_length} ${base_width} ${base_height}; visual mesh filename=package://sam_bot_description/meshes/robot_base.stl
